File: TurtleSensor.sch (KiCad schematic (older format))
At the start: 15 parts, among them IC1 ATMEGA328P-A, J2 FTDIConnector, U1 SI7021, U2 M24512

Commit message: before copper fill
Parts:
- 32KHz1: footprint footprints:2-SMD -> Resistors_SMD:R_0805_HandSoldering
- renumbered 2k to 2k1
Connections:
- net SCK: now also D1.2 (A)
- net at IC1.13 ((PCINT1/OC1A)PB1): no longer D1.2 (A)
Changed lines of the file:
@@
 Wire Wire Line
 	5200 1650 5100 1650
-Wire Wire Line
-	4700 1650 4300 1650
 $Comp
 L Crystal 32KHz1
@@
 F 0 "32KHz1" H 5200 2350 50  0000 C CNN
 F 1 "Crystal" H 5200 2050 50  0000 C CNN
-F 2 "footprints:2-SMD" H 5200 2200 50  0001 C CNN
+F 2 "Resistors_SMD:R_0805_HandSoldering" H 5200 2200 50  0001 C CNN
 F 3 "" H 5200 2200 50  0000 C CNN
 	1    5200 2200
@@
 	8300 2000 8300 2100
 $Comp
-L R 2k
+L R 2k1
 U 1 1 57C323B4
 P 3950 6150
-F 0 "2k" V 4030 6150 50  0000 C CNN
+F 0 "2k1" V 4030 6150 50  0000 C CNN
 F 1 "R" V 3950 6150 50  0000 C CNN
-F 2 "" V 3880 6150 50  0000 C CNN
+F 2 "" V 3880 6150 50  0001 C CNN
 F 3 "" H 3950 6150 50  0000 C CNN
 	1    3950 6150
@@
 	3950 6300 3950 6400
 Connection ~ 3950 6400
+Wire Wire Line
+	4700 1650 4500 1650
+Text Label 4500 1650 0    60   ~ 0
+SCK
 $EndSCHEMATC

Commit message: rerouted power
Parts:
- removed C1: 10µF, Capacitors_SMD:C_0805_HandSoldering, symbol CP
- added C1: 0.1µF, Capacitors_SMD:C_0805_HandSoldering, symbol C
- added C5: 10µF, Capacitors_SMD:C_0805_HandSoldering, symbol C
- 10k1: renamed from 2k1; value R -> 10k; footprint (none) -> Resistors_SMD:R_0805_HandSoldering
- 32kHz1: renamed from 32KHz1; value Crystal -> TXC 9HT11-32.768KDZF-T
- BT1: value Battery -> 534-3039; symbol Battery -> Battery-RESCUE-TurtleSensor
- C3: renamed from 22pF1; value C -> 12.5pF
- C4: renamed from 22pF2; value C -> 12.5pF
- D1: value LED -> 5988110107F; symbol LED -> LED-RESCUE-TurtleSensor
- IC1: value ATMEGA328P-A -> ATMEGA328PB-A
- J1: renamed from J2; footprint Pin_Headers:Pin_Header_Straight_1x06 -> Pin_Headers:Pin_Header_Straight_1x06_Pitch2.54mm
- R1: value 470 -> 33Ω
- R2, R3: value 4k -> 4k7
- U1: value SI7021 -> SI7021-A20-GM1R
- U2: value M24512 -> M24M01-RMN6TP
Connections:
- net +BATT: now also C1.1, C5.1
- net GND: now also C1.2, C5.2
- net RX: now also IC1.32 ((PCINT18/INT0)PD2)
- net ~CS renamed ~SS
- no-connect marks 14 -> 13
Other:
- moved on the sheet: 10k1, C2
Changed lines of the file:
@@
 $EndDescr
 $Comp
-L Battery BT1
+L Battery-RESCUE-TurtleSensor BT1
 U 1 1 5622E668
 P 1100 2750
 F 0 "BT1" H 1200 2800 50  0000 L CNN
-F 1 "Battery" H 1200 2700 50  0000 L CNN
+F 1 "534-3039" H 1200 2700 50  0000 L CNN
 F 2 "footprints:2477Holder" V 1100 2790 60  0001 C CNN
 F 3 "" V 1100 2790 60  0000 C CNN
@@
 Wire Wire Line
 	1100 3650 1100 2900
-$Comp
-L CP C1
-U 1 1 5622E715
-P 2150 2600
-F 0 "C1" H 2175 2700 50  0000 L CNN
-F 1 "10µF" H 2175 2500 50  0000 L CNN
-F 2 "Capacitors_SMD:C_0805_HandSoldering" H 2188 2450 30  0001 C CNN
-F 3 "" H 2150 2600 60  0000 C CNN
-	1    2150 2600
-	1    0    0    -1
-$EndComp
 Connection ~ 2150 1850
 Wire Wire Line
@@
 Connection ~ 2150 3750
 $Comp
-L LED D1
+L LED-RESCUE-TurtleSensor D1
 U 1 1 5622E8A4
 P 4900 1650
 F 0 "D1" H 4900 1750 50  0000 C CNN
-F 1 "LED" H 4900 1550 50  0000 C CNN
+F 1 "5988110107F" H 4900 1550 50  0000 C CNN
 F 2 "LEDs:LED_0805" H 4900 1650 60  0001 C CNN
-F 3 "" H 4900 1650 60  0000 C CNN
+F 3 "http://www.newark.com/dialight/5988110107f/led-red-1-25mm-x-1-4mm-40mcd-642nm/dp/75R0581" H 4900 1650 60  0000 C CNN
 	1    4900 1650
 	-1   0    0    1
@@
 P 5350 1650
 F 0 "R1" V 5430 1650 50  0000 C CNN
-F 1 "470" V 5350 1650 50  0000 C CNN
+F 1 "33Ω" V 5350 1650 50  0000 C CNN
 F 2 "Resistors_SMD:R_0805_HandSoldering" V 5280 1650 30  0001 C CNN
 F 3 "" H 5350 1650 30  0000 C CNN
@@
 	5200 1650 5100 1650
 $Comp
-L Crystal 32KHz1
+L Crystal 32kHz1
 U 1 1 56B6E109
 P 5200 2200
-F 0 "32KHz1" H 5200 2350 50  0000 C CNN
-F 1 "Crystal" H 5200 2050 50  0000 C CNN
+F 0 "32kHz1" H 5200 2350 50  0000 C CNN
+F 1 "TXC 9HT11-32.768KDZF-T" H 5200 2050 50  0000 C CNN
 F 2 "Resistors_SMD:R_0805_HandSoldering" H 5200 2200 50  0001 C CNN
-F 3 "" H 5200 2200 50  0000 C CNN
+F 3 "https://octopart.com/9ht11-32.768kdzf-t-txc-18803093" H 5200 2200 50  0000 C CNN
 	1    5200 2200
 	0    1    1    0
 $EndComp
 $Comp
-L C 22pF1
+L C C3
 U 1 1 56B6E156
 P 5650 2050
-F 0 "22pF1" H 5675 2150 50  0000 L CNN
-F 1 "C" H 5675 1950 50  0000 L CNN
+F 0 "C3" H 5675 2150 50  0000 L CNN
+F 1 "12.5pF" H 5675 1950 50  0000 L CNN
 F 2 "Capacitors_SMD:C_0805_HandSoldering" H 5688 1900 50  0001 C CNN
 F 3 "" H 5650 2050 50  0000 C CNN
@@
 $EndComp
 $Comp
-L C 22pF2
+L C C4
 U 1 1 56B6E19B
 P 5650 2350
-F 0 "22pF2" H 5675 2450 50  0000 L CNN
-F 1 "C" H 5675 2250 50  0000 L CNN
+F 0 "C4" H 5675 2450 50  0000 L CNN
+F 1 "12.5pF" H 5675 2250 50  0000 L CNN
 F 2 "Capacitors_SMD:C_0805_HandSoldering" H 5688 2200 50  0001 C CNN
 F 3 "" H 5650 2350 50  0000 C CNN
@@
 	2150 2150 2400 2150
 Connection ~ 2150 2150
-Text Label 5250 3500 0    60   ~ 0
-~CS
-Text Label 5700 3500 0    60   ~ 0
-~SS
-Wire Wire Line
-	5700 3500 5250 3500
 Wire Wire Line
 	2400 3850 2150 3850
@@
 ~RST
 $Comp
-L FTDIConnector J2
+L FTDIConnector J1
 U 1 1 56DB7438
 P 5550 6000
-F 0 "J2" H 5300 6600 60  0000 C CNN
+F 0 "J1" H 5300 6600 60  0000 C CNN
 F 1 "FTDIConnector" H 5350 5350 60  0000 C CNN
-F 2 "Pin_Headers:Pin_Header_Straight_1x06" H 5550 5650 60  0001 C CNN
+F 2 "Pin_Headers:Pin_Header_Straight_1x06_Pitch2.54mm" H 5550 5650 60  0001 C CNN
 F 3 "" H 5550 5650 60  0000 C CNN
 	1    5550 6000
@@
 	5000 6250 4700 6250
 Wire Wire Line
-	4400 6400 5000 6400
-Text Label 3700 6400 0    60   ~ 0
+	4100 6400 5000 6400
+Text Label 3400 6400 0    60   ~ 0
 ~RST
 Text Label 4700 6250 0    60   ~ 0
@@
 TX
 Wire Wire Line
-	3950 5950 5000 5950
-Wire Wire Line
 	4550 6550 4550 5650
 Wire Wire Line
 	4550 5650 5000 5650
-Wire Wire Line
-	4400 5500 4400 5950
 NoConn ~ 5000 5800
 NoConn ~ 4300 1550
@@
 NoConn ~ 4300 2600
 NoConn ~ 4300 2700
-NoConn ~ 4300 3350
 NoConn ~ 4300 3450
 NoConn ~ 4300 3550
@@
 L C C2
 U 1 1 56DB8C77
-P 4250 6400
-F 0 "C2" H 4275 6500 50  0000 L CNN
-F 1 "0.1uF" H 4275 6300 50  0000 L CNN
-F 2 "Capacitors_SMD:C_0805_HandSoldering" H 4288 6250 50  0001 C CNN
-F 3 "" H 4250 6400 50  0000 C CNN
-	1    4250 6400
+P 3950 6400
+F 0 "C2" H 3975 6500 50  0000 L CNN
+F 1 "0.1uF" H 3975 6300 50  0000 L CNN
+F 2 "Capacitors_SMD:C_0805_HandSoldering" H 3988 6250 50  0001 C CNN
+F 3 "" H 3950 6400 50  0000 C CNN
+	1    3950 6400
 	0    1    1    0
 $EndComp
 Wire Wire Line
-	4100 6400 3700 6400
+	3400 6400 3800 6400
 $Comp
 L SI7021 U1
@@
 P 6850 2350
 F 0 "U1" H 6550 2570 50  0000 L CNN
-F 1 "SI7021" H 6550 2060 50  0000 L CNN
+F 1 "SI7021-A20-GM1R" H 6550 2060 50  0000 L CNN
 F 2 "SI7021:DFN-6%2f3MM" H 6850 2350 50  0001 L CNN
-F 3 "" H 6850 2350 60  0000 C CNN
+F 3 "https://www.silabs.com/Support%20Documents%2FTechnicalDocs%2FSi7021-A20.pdf" H 6850 2350 60  0000 C CNN
 	1    6850 2350
 	1    0    0    -1
@@
 P 3300 2650
 F 0 "IC1" H 2550 3900 50  0000 L BNN
-F 1 "ATMEGA328P-A" H 3700 1250 50  0000 L BNN
+F 1 "ATMEGA328PB-A" H 3700 1250 50  0000 L BNN
 F 2 "Housings_QFP:TQFP-32_7x7mm_Pitch0.8mm" H 3300 2650 50  0000 C CIN
-F 3 "" H 3300 2650 50  0000 C CNN
+F 3 "http://www.atmel.com/Images/Atmel-42397-8-bit-AVR-Microcontroller-ATmega328PB_Datasheet.pdf" H 3300 2650 50  0000 C CNN
 	1    3300 2650
 	1    0    0    -1
@@
 P 7400 3600
 F 0 "U2" H 7450 3950 60  0000 C CNN
-F 1 "M24512" H 7400 3450 60  0000 C CNN
+F 1 "M24M01-RMN6TP" H 7400 3450 60  0000 C CNN
 F 2 "SMD_Packages:SOIC-8-N" H 7400 3600 60  0001 C CNN
-F 3 "" H 7400 3600 60  0000 C CNN
+F 3 "www.st.com/resource/en/datasheet/m24m01-df.pdf" H 7400 3600 60  0000 C CNN
 	1    7400 3600
 	1    0    0    -1
@@
 P 8300 1850
 F 0 "R2" V 8380 1850 50  0000 C CNN
-F 1 "4k" V 8300 1850 50  0000 C CNN
+F 1 "4k7" V 8300 1850 50  0000 C CNN
 F 2 "Resistors_SMD:R_0805_HandSoldering" V 8230 1850 50  0001 C CNN
 F 3 "" H 8300 1850 50  0000 C CNN
@@
 P 8700 1850
 F 0 "R3" V 8780 1850 50  0000 C CNN
-F 1 "4k" V 8700 1850 50  0000 C CNN
+F 1 "4k7" V 8700 1850 50  0000 C CNN
 F 2 "Resistors_SMD:R_0805_HandSoldering" V 8630 1850 50  0001 C CNN
 F 3 "" H 8700 1850 50  0000 C CNN
@@
 	8300 2000 8300 2100
 $Comp
-L R 2k1
+L R 10k1
 U 1 1 57C323B4
-P 3950 6150
-F 0 "2k1" V 4030 6150 50  0000 C CNN
-F 1 "R" V 3950 6150 50  0000 C CNN
-F 2 "" V 3880 6150 50  0001 C CNN
-F 3 "" H 3950 6150 50  0000 C CNN
-	1    3950 6150
-	1    0    0    -1
-$EndComp
-Connection ~ 4400 5950
-Wire Wire Line
-	3950 5950 3950 6000
-Wire Wire Line
-	3950 6300 3950 6400
-Connection ~ 3950 6400
+P 3950 5950
+F 0 "10k1" V 4030 5950 50  0000 C CNN
+F 1 "10k" V 3950 5950 50  0000 C CNN
+F 2 "Resistors_SMD:R_0805_HandSoldering" V 3880 5950 50  0001 C CNN
+F 3 "" H 3950 5950 50  0000 C CNN
+	1    3950 5950
+	0    1    1    0
+$EndComp
 Wire Wire Line
 	4700 1650 4500 1650
 Text Label 4500 1650 0    60   ~ 0
 SCK
+$Comp
+L C C5
+U 1 1 57FE8071
+P 2150 2600
+F 0 "C5" H 2175 2700 50  0000 L CNN
+F 1 "10µF" H 2175 2500 50  0000 L CNN
+F 2 "Capacitors_SMD:C_0805_HandSoldering" H 2188 2450 50  0001 C CNN
+F 3 "" H 2150 2600 50  0000 C CNN
+	1    2150 2600
+	1    0    0    -1
+$EndComp
+$Comp
+L C C1
+U 1 1 57FE81CA
+P 1850 2600
+F 0 "C1" H 1875 2700 50  0000 L CNN
+F 1 "0.1µF" H 1875 2500 50  0000 L CNN
+F 2 "Capacitors_SMD:C_0805_HandSoldering" H 1888 2450 50  0001 C CNN
+F 3 "" H 1850 2600 50  0000 C CNN
+	1    1850 2600
+	1    0    0    -1
+$EndComp
+Wire Wire Line
+	1850 2750 1850 3650
+Connection ~ 1850 3650
+Wire Wire Line
+	1850 2450 1850 1550
+Connection ~ 1850 1550
+Wire Wire Line
+	4100 5950 5000 5950
+Wire Wire Line
+	4300 3350 4500 3350
+Text Label 4500 3350 0    60   ~ 0
+RX
+Wire Wire Line
+	3800 5950 3700 5950
+Wire Wire Line
+	3700 5950 3700 6400
+Connection ~ 3700 6400
+Wire Wire Line
+	4400 5500 4400 5950
+Connection ~ 4400 5950
 $EndSCHEMATC
